Commit message: Completed robot enhancements.

File: projects/go_chase_it/my_robot/urdf/my_robot.xacro (robot description, xacro)
@@ -55,3 +55,65 @@
     </visual>
   </link>
+  <joint name="left_wheel_joint" type="continuous">
+    <origin xyz="0 .15 0" rpy="0 0 0"/>
+    <parent link="chassis"/>
+    <child link="left_wheel"/>
+    <axis xyz="0 1 0" rpy="0 0 0"/>
+    <limit effort="10000" velocity="1000"/>
+    <dynamics damping="1.0" friction="1.0"/>
+  </joint>
+  <link name="left_wheel">
+    <inertial>
+      <mass value="5.0"/>
+      <origin xyz="0 0 0" rpy="0 0 0"/>
+      <inertia
+        ixx="0.1" ixy="0" ixz="0"
+        iyy="0.1" iyz="0"
+        izz="0.1"
+      />
+    </inertial>
+    <collision>
+      <origin xyz="0 0 0" rpy="0 1.5707 1.5707"/>
+      <geometry>
+        <cylinder radius=".1" length=".05"/>
+      </geometry>
+    </collision>
+    <visual>
+      <origin xyz="0 0 0" rpy="0 1.5707 1.5707"/>
+      <geometry>
+        <cylinder radius=".1" length=".05"/>
+      </geometry>
+    </visual>
+  </link>
+  <joint name="right_wheel_joint" type="continuous">
+    <origin xyz="0 -.15 0" rpy="0 0 0"/>
+    <parent link="chassis"/>
+    <child link="right_wheel"/>
+    <axis xyz="0 1 0" rpy="0 0 0"/>
+    <limit effort="10000" velocity="1000"/>
+    <dynamics damping="1.0" friction="1.0"/>
+  </joint>
+  <link name="right_wheel">
+    <inertial>
+      <mass value="5.0"/>
+      <origin xyz="0 0 0" rpy="0 0 0"/>
+      <inertia
+        ixx="0.1" ixy="0" ixz="0"
+        iyy="0.1" iyz="0"
+        izz="0.1"
+      />
+    </inertial>
+    <collision>
+      <origin xyz="0 0 0" rpy="0 1.5707 1.5707"/>
+      <geometry>
+        <cylinder radius=".1" length=".05"/>
+      </geometry>
+    </collision>
+    <visual>
+      <origin xyz="0 0 0" rpy="0 1.5707 1.5707"/>
+      <geometry>
+        <cylinder radius=".1" length=".05"/>
+      </geometry>
+    </visual>
+  </link>
 </robot>

Commit message: Added sensor models to robot and added Gazebo colors.

File: projects/go_chase_it/my_robot/urdf/my_robot.xacro (robot description, xacro)
@@ -117,3 +117,74 @@
     </visual>
   </link>
+  <joint name="camera_joint" type="fixed">
+    <origin xyz=".2 0 0" rpy="0 0 0"/>
+    <parent link="chassis"/>
+    <child link="camera"/>
+    <axis xyz="0 1 0" rpy="0 0 0"/>
+  </joint>
+  <link name="camera">
+    <inertial>
+      <mass value=".1"/>
+      <origin xyz="0 0 0" rpy="0 0 0"/>
+      <inertia
+        ixx="1e-6" ixy="0" ixz="0"
+        iyy="1e-6" iyz="0"
+        izz="1e-6"
+      />
+    </inertial>
+    <collision>
+      <origin xyz="0 0 0" rpy="0 0 0"/>
+      <geometry>
+        <box size=".05 .05 .05"/>
+      </geometry>
+    </collision>
+    <visual>
+      <origin xyz="0 0 0" rpy="0 0 0"/>
+      <geometry>
+        <box size=".05 .05 .05"/>
+      </geometry>
+    </visual>
+  </link>
+  <joint name="hokuyo_joint" type="fixed">
+    <origin xyz=".15 0 .1" rpy="0 0 0"/>
+    <parent link="chassis"/>
+    <child link="hokuyo"/>
+    <axis xyz="0 1 0" rpy="0 0 0"/>
+  </joint>
+  <link name="hokuyo">
+    <inertial>
+      <mass value="1e-5"/>
+      <origin xyz="0 0 0" rpy="0 0 0"/>
+      <inertia
+        ixx="1e-6" ixy="0" ixz="0"
+        iyy="1e-6" iyz="0"
+        izz="1e-6"
+      />
+    </inertial>
+    <collision>
+      <origin xyz="0 0 0" rpy="0 0 0"/>
+      <geometry>
+        <box size=".1 .1 .1"/>
+      </geometry>
+    </collision>
+    <visual>
+      <origin xyz="0 0 0" rpy="0 0 0"/>
+      <geometry>
+        <mesh filename="package://my_robot/meshes/hokuyo.dae"/>
+      </geometry>
+    </visual>
+  </link>
+  <!--Add colors for Gazebo-->
+  <gazebo reference="left_wheel">
+    <material>Gazebo/Black</material>
+  </gazebo>
+  <gazebo reference="right_wheel">
+    <material>Gazebo/Black</material>
+  </gazebo>
+  <gazebo reference="chassis">
+    <material>Gazebo/Yellow</material>
+  </gazebo>
+  <gazebo reference="camera">
+    <material>Gazebo/Black</material>
+  </gazebo>
 </robot>

Commit message: Added states to process image node so service called only when update needed. Relocated color specifications in URDF files.

File: projects/go_chase_it/my_robot/urdf/my_robot.xacro (robot description, xacro)
@@ -176,16 +176,3 @@
     </visual>
   </link>
-  <!--Add colors for Gazebo-->
-  <gazebo reference="left_wheel">
-    <material>Gazebo/Black</material>
-  </gazebo>
-  <gazebo reference="right_wheel">
-    <material>Gazebo/Black</material>
-  </gazebo>
-  <gazebo reference="chassis">
-    <material>Gazebo/Yellow</material>
-  </gazebo>
-  <gazebo reference="camera">
-    <material>Gazebo/Black</material>
-  </gazebo>
 </robot>
